File: hardware/AO-Horizon/AO-Horizon.kicad_sch (KiCad schematic)
At the start: 0 parts

Commit message: Update AO-Horizon.kicad_sch
Other:
- added sheet Block Diagram (block_diagram.kicad_sch)
- added sheet Revision History (revision_history.kicad_sch)
- added sheet Top (top_hierarchical.kicad_sch)
- note added: "${RELEASE_DATE}"
- note added: "......"
- note added: "1"
- note added: "2"
- note added: "3"
- note added: "4"
- note added: "5"
- note added: "6"
- note added: "7"
- note added: "8"
- note added: "9"
- note added: "A"
- note added: "B"
- note added: "Block Diagram"
- note added: "Bottom View"
- note added: "C"
- note added: "D"
- note added: "E"
- note added: "Flight Controller on STM32H7 Series"
- note added: "General Note"
- note added: "Legend"
- note added: "Power Supplies"
- note added: "Project Overview"
- note added: "Rev: ${REVISION}"
- note added: "Revision History"
- note added: "Table of Contents"
- note added: "Text to be added to silkscreen."
- note added: "The Horizon"
- note added: "Top Hierarchical View"
- note added: "Top View"
- note added: "Warning Note"
