File: hardware/AO-Horizon/power_supplies.kicad_sch (KiCad schematic)
At the start: 44 parts

Commit message: feat(schematic): replace the eFuse with TPS259251DRC and rework the buck input
Replace the TPS16412DRC eFuse and its OVP, IOCP/IMON, IDLY and fault
LED parts with a TPS259251DRC (DEC-026): EN/UVLO 1M to +VIN, ILIM 45k3,
dV/dT 1n. Feed the TPS62142 from +5V through a 0.33 uH inductor instead
of the ferrite bead, add the AVIN 100n, use a 3.3 uH PCR0420 buck
inductor, and set the LDO NR capacitor to 10n.

Put the TPS25925x and TPS25926x symbols in the BOM and on the board,
add an L_0603_1608Metric footprint, and drop unused capacitor, inductor
and JST ZH library items.

Parts are unannotated. eFuse values not checked against TI data. ERC
not run.

Co-Authored-By: Claude Opus 5.5 <noreply@anthropic.com>
Parts:
- removed C? (x3): 100n, 0_Capacitor_SMD:C_0402_1005Metric_NomDensity, symbol Device:C
- removed C? (x4): 10u, 0_Capacitor_SMD:C_0805_2012Metric_NomDensity, symbol Device:C
- removed C? (x2): 10n, symbol Device:C
- removed D?: D_Zener, symbol Device:D_Zener
- removed D?: LTST-C191KRKT, 0_LED_SMD:LED_0603_1608Metric, symbol Device:LED
- removed L?: FerriteBead, symbol Device:FerriteBead
- removed R? (x2): 1k, symbol Device:R
- removed R? (x3): 10k, symbol Device:R
- removed R?: 6k49, symbol Device:R
- removed R?: 29k4, symbol Device:R
- removed U?: TPS16412DRC, 0_Package_SON:Texas_VSON-10-1EP_3x3mm_P0.5mm_EP1.65x2.4mm_ThermalVias, symbol 0_Protection_eFuse:TPS16412DRC
- removed U?: TPS259241DRC, 0_Package_SON:Texas_VSON-10-1EP_3x3mm_P0.5mm_EP1.65x2.4mm_ThermalVias, symbol 0_Protection_eFuse:TPS25924xDRC
- added C? (x2): 100n, 0_Capacitor_SMD:C_0402_1005Metric_NomDensity, symbol Device:C
- added C?: 10n, symbol Device:C
- added C?: 10u, 0_Capacitor_SMD:C_0805_2012Metric_NomDensity, symbol Device:C
- added L?: ASMPH-0603-R33M-T, 0_Inductor_SMD:L_0603_1608Metric, symbol Device:L
- added U?: TPS259251DRC, 0_Package_SON:Texas_VSON-10-1EP_3x3mm_P0.5mm_EP1.65x2.4mm_ThermalVias, symbol 0_Protection_eFuse:TPS25925xDRC
- C?: value 10n -> 1n
- R?: value 10k -> 1Meg
- R?: value 43k2 -> 45k3
Connections:
- net +5V: now also C?.1, C?.1, L?.1, U?.6 (OUT), U?.7 (OUT), U?.8 (OUT)
- net +5V_BUCK: now also L?.2
- net +VIN: now also C?.1, C?.1, U?.3 (VIN), U?.4 (VIN), U?.5 (VIN); no longer C?.1
- net FUSE_EN: now also R?.2, U?.2 (EN/UVLO)
- net FUSE_ILIM: now also R?.1, U?.10 (ILIM)
- net FUSE_dVdT: now also C?.1, U?.1 (dV/dT)
- net GND: now also C?.2, C?.2, C?.2, C?.2, U?.11 (GND)
- net LDO_FB: now also C?.1
Other:
- note added: "330nH 150mR"
- note added: "Fast-trip Overload Current limit"
- note added: "I_{FASTRIP} = 1.6 x I_{ILIM} I_{FASTRIP} = 1.6 x 2.05A = 3.28A Device shutdown when : I_{OUT} > I_{FASTRIP}"
- note added: "I_{INRUSH} = 20uF x (5V / 350us) I_{INRUSH} = 286mA"
- note added: "I_{INRUSH} = 20uF x (5V / 5.35ms) I_{INRUSH} = 18.7mA"
- note added: "Inrush current drawn by C_{OUT}"
- note added: "Output Voltage Ramp Time (TdVdT)"
- note added: "P_{D(Load)} = V_{IN}^{2}/(6 x R_{Load}) P_{D(Load)} = 5^{2}/(6 x 5/0.5) #~0.5A Load P_{D(Load)} = 0.42W P_{D(INRUSH,1)} = 0.5 x 5V x 286mA = 715mW P_{D(INRUSH,2)} = 0.5 x 5V x 18.7mA = 46.8mW P_{D(STARTUP)} = P_{D(INRUSH)} + P_{D(Load)} P_{D(STARTUP,1)} = 1.14W @ NC P_{D(STARTUP,2)} = 0.47W @ 1nF"
- note added: "Power Dissipation during Start-Up"
- note added: "Recovery from Short Circuit"
- note added: "TPS2592x1 : Auto-retry V_{IN} = 5 V about 100 - 120ms."
- note added: "TdVdT = 10e6 x V_{IN}(C_{dVdT} + 70pF) = 10e6 x 5V(1nF + 70pF) = 350us. = 10e6 x 5V(0 + 70pF) = 5.35ms."
- note added: "The R_{ILIM} resistor at the ILIM pin R_{ILIM} = (I_{ILIM} - 0.7) / 3e-5 R_{ILIM} = (2.05A - 0.7) / 3e-5 R_{ILIM} = 45k choose R=45.3kΩ"
- note added: "UVLO threshold, rising : 4.3V @ Vin UVLO hysteresis : 5% : 4.1V @ Vin EN threshold voltage, rising : 1.4V EN threshold voltage, falling : 1.35V"
- note added: "Undervoltage Lockout"
- note removed: "Action: I_{LIM} ≤ I_{OUT} < I_{OCP} : Provides current up to I_{OCP} and then limit to I_{LIM} I_{OCP} ≤ I_{OUT} < I_{Ifast-trip} : Limits current to ILIM I_{Ifast-trip} ≤ I_{OUT} < I_{SCP} : Turns off the internal FET"
- note removed: "Active Current Limiting"
- note removed: "Blanking Time (t_{IDLY})"
- note removed: "C_{dVdT} = 100e-6 / SR SR = I_{Inrush} / C_{OUT} C_{dVdT} = 100e-6 /(0.5A / ~50uF) C_{dVdT} = (10nF)"
- note removed: "Do not connect the EN pin more than 5V."
- note removed: "EN rising TH : 1.40V (typ.) EN falling TH : 1.35V (typ.) Ru = 29.4kΩ, Rd = 10kΩ Action: Device turns off : V_{IN} above 6.03V and Device Reset : V_{IN} below 5.5V if not use, Connect OVP pin to GND"
- note removed: "I_{LIM} = 0.984A x 10k / (R_{LIM}) I_{LIM} = 0.984A x 10k / (6.49kΩ) I_{LIM} = 1.516A"
- note removed: "I_{OCP} = 2.25A x 7.32k / (R_{IOCP}) I_{OCP} = 2.25A x 7.32k / (10kΩ) I_{OCP} = 1.647A I_{Ifast-trip} = 1.9 x I_{OCP} = 3.13A I_{SCP} = 6.7A (typ)"
- note removed: "Inrush Current Control"
- note removed: "OVP rising th : 1.53V (typ.) OVP falling th : 1.40V (typ.) Ru = 29.4kΩ, Rd = 10kΩ Action: Device turns off : V_{IN} above 6.03V and Device Reset : V_{IN} below 5.5V if not use, Connect OVP pin to GND"
- note removed: "Output Slew Rate Control"
- note removed: "Overcurrent Protection"
- note removed: "Overvoltage Protection Setpoint"
- note removed: "The R_{ILIM} resistor at the ILIM pin R_{ILIM} = (I_{ILIM} - 0.7) / 3e-5 R_{ILIM} = (2A - 0.7) / 3e-5 R_{ILIM} = 43.3k choose R=43.2kΩ"
- note removed: "Undervoltage Lockout Setpoint"
- note removed: "Vf = 1.8V IV = 180mcd @20mA 9mcd @ 1mA"
- note removed: "dVdt = 100e-6 / C_{dVdT} = 100e-6 / (10nF) = 10e3 V/s Vout = 5V, dVdt = 10e3V/s Vout rising = 500us."
- note removed: "sink current into FLT pin is less than 3mA"
- note removed: "t_{IDLY} = (6.5ms/12nF) x (C_{DLY}) t_{IDLY} = (6.5ms/12nF) x (10nF) Blanking time before current limiting = 5.42ms."
- moved on the sheet: C?, CN?, R?
