File: hardware/AO-Horizon/AO-Horizon.kicad_pcb (KiCad board)
At the start: 2 copper layers, 0 parts

Commit message: feat: TPS259251DRC eFuse (DEC-026), spec 0.18 and power view update (#30)
* docs(readme): simplify workflow diagram explanation

Mark DRAFT as under review, sync CHECK label, and add a colour key in README and template.

Co-Authored-By: Claude Sonnet 5.5 <noreply@anthropic.com>

* Update settings.json

* change spec file name

* update git-workflow skill

* change skill name by add hw-*

* docs: update AeroOptix-Horizon hardware spec

* docs: consolidate hardware handoff into checklist

* Update CLAUDE.md

* Update CLAUDE.md

* Update CLAUDE.md

* feat(hooks): replace protect hook with rule-based v2

Move file-protection rules into hooks/protect.json (allow > deny > ask)
and use ask for editable-with-approval files instead of a hard block.
Bash/PowerShell checks now inspect write targets, not any mention of a
protected path. Align settings.json permissions and drop the old hook.

Co-Authored-By: Claude Sonnet 5.5 <noreply@anthropic.com>

* docs: update CLAUDE.md for protection tiers and skill names

Describe the ask/deny protection rules, the v2 hook and protect.json,
and fix stale skill and template names.

Co-Authored-By: Claude Sonnet 5.5 <noreply@anthropic.com>

* Update .gitignore

* Update .gitignore

* Update .gitignore

* del skills

* Update engineering.md

* Update git-workflow.md

* Update hardware-workflow.md

* Update settings.json

* Update pull_request_template.md

* Update .gitignore

* Update .gitignore

* Delete SKILL.md

* Delete SKILL.md

* Update .gitignore

* add git-workflow skill

* Update CLAUDE.md

* Update protect.json

* Update settings.json

* Create MEMORY.md

* feat(agents): add codex-hw-delegate for bounded Codex tasks

Add a project agent that delegates one small, read-only-by-default task
to Codex CLI. It gates trivial or ambiguous requests, refuses PDF and
KiCad file contents, never mutates git, cross-checks Codex output and
returns a fixed report format.

Co-Authored-By: Claude Sonnet 5.5 <noreply@anthropic.com>

* fix(hooks): res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
Other:
- board text added: "Board Specifications"
- board text added: "Bottom Assembly (Scale 1:1)"
- board text added: "Bottom Dimension (Scale 1:1)"
- board text added: "Bottom Testpoint (Scale 1:1)"
- board text added: "Top Assembly (Scale 1:1)"
- board text added: "Top Dimension (Scale 1:1)"
- board text added: "Top Testpoint (Scale 1:1)"

Commit message: feat: close the power sheet capture (spec 0.19, DEC-027, DEC-028) (#31)
* docs(readme): simplify workflow diagram explanation

Mark DRAFT as under review, sync CHECK label, and add a colour key in README and template.

Co-Authored-By: Claude Sonnet 5.5 <noreply@anthropic.com>

* Update settings.json

* change spec file name

* update git-workflow skill

* change skill name by add hw-*

* docs: update AeroOptix-Horizon hardware spec

* docs: consolidate hardware handoff into checklist

* Update CLAUDE.md

* Update CLAUDE.md

* Update CLAUDE.md

* feat(hooks): replace protect hook with rule-based v2

Move file-protection rules into hooks/protect.json (allow > deny > ask)
and use ask for editable-with-approval files instead of a hard block.
Bash/PowerShell checks now inspect write targets, not any mention of a
protected path. Align settings.json permissions and drop the old hook.

Co-Authored-By: Claude Sonnet 5.5 <noreply@anthropic.com>

* docs: update CLAUDE.md for protection tiers and skill names

Describe the ask/deny protection rules, the v2 hook and protect.json,
and fix stale skill and template names.

Co-Authored-By: Claude Sonnet 5.5 <noreply@anthropic.com>

* Update .gitignore

* Update .gitignore

* Update .gitignore

* del skills

* Update engineering.md

* Update git-workflow.md

* Update hardware-workflow.md

* Update settings.json

* Update pull_request_template.md

* Update .gitignore

* Update .gitignore

* Delete SKILL.md

* Delete SKILL.md

* Update .gitignore

* add git-workflow skill

* Update CLAUDE.md

* Update protect.json

* Update settings.json

* Create MEMORY.md

* feat(agents): add codex-hw-delegate for bounded Codex tasks

Add a project agent that delegates one small, read-only-by-default task
to Codex CLI. It gates trivial or ambiguous requests, refuses PDF and
KiCad file contents, never mutates git, cross-checks Codex output and
returns a fixed report format.

Co-Authored-By: Claude Sonnet 5.5 <noreply@anthropic.com>

* fix(hooks): resol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
Other:
- board outline added: 27 x 29 mm
Changed lines of the file:
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@@
 	(property "AUTHOR" "NATCHANON THUENTHAM")
 	(property "EX_PAGE" "1")
+	(property "KICAD_VERSION" "KiCad E.D.A 10.0.8")
 	(property "PCB_DRAWING_DATE" "")
 	(property "PCB_DRAWING_NAME" "")
 	(property "PCB_REVIEW_DATE" "")
 	(property "PCB_REVIEW_NAME" "")
-	(property "PROJECT_ID" "NP-AO-2601")
+	(property "PROJECT_ID" "NP-AO-2601-V1-0")
 	(property "PROJECT_NAME" "AeroOptix - Horizon")
-	(property "RELEASE_DATE" "DD MM 202X")
+	(property "RELEASE_DATE" "")
 	(property "SCH_DRAWING_DATE" "")
 	(property "SCH_DRAWING_NAME" "")
 	(property "SCH_REVIEW_DATE" "")
 	(property "SCH_REVIEW_NAME" "")
+	(gr_rect
+		(start 144 81)
+		(end 171 110)
+		(stroke
+			(width 0.05)
+			(type default)
+		)
+		(fill no)
+		(layer "Edge.Cuts")
+	)
 	(gr_text "Top Testpoint (Scale 1:1)"
 		(at 150 22 0)
